File: hardware/pcb/counter/counter.kicad_pcb (KiCad board)
At the start: 4 copper layers, 62.2 x 21.6 mm, 54 parts, among them J2 Control, J3 Sync, J4 + Power -, J5 Address Bus, J6 NC, U1 74HC161, U10 74HC173, U2 74HC173, U5 74HC161, U6 74HC173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

Commit message: PC finishing touches
Parts:
- added D17: OUT, LED_SMD:LED_0805_2012Metric_Pad1.15x1.40mm_HandSolder, F.Cu at (42.8, 46.8)
- added D18: LOAD, LED_SMD:LED_0805_2012Metric_Pad1.15x1.40mm_HandSolder, F.Cu at (42.8, 49.1)
- added D19: COUNT, LED_SMD:LED_0805_2012Metric_Pad1.15x1.40mm_HandSolder, F.Cu at (42.8, 51.3)
- added R17: 330, Resistor_SMD:R_0805_2012Metric_Pad1.20x1.40mm_HandSolder, B.Cu at (40.8, 46.8)
- added R18: 10K, Resistor_SMD:R_0805_2012Metric_Pad1.20x1.40mm_HandSolder, B.Cu at (36.8, 52.2)
- added R19: 330, Resistor_SMD:R_0805_2012Metric_Pad1.20x1.40mm_HandSolder, B.Cu at (40.8, 49.0)
- added R20: 10K, Resistor_SMD:R_0805_2012Metric_Pad1.20x1.40mm_HandSolder, B.Cu at (39.4, 52.2)
- added R21: 330, Resistor_SMD:R_0805_2012Metric_Pad1.20x1.40mm_HandSolder, B.Cu at (42.9, 51.3)
- added R22: 10K, Resistor_SMD:R_0805_2012Metric_Pad1.20x1.40mm_HandSolder, B.Cu at (48.5, 55.9)
- added R23: 100K, Resistor_SMD:R_0805_2012Metric_Pad1.20x1.40mm_HandSolder, F.Cu at (71.5, 55.9)
- added R24: 100K, Resistor_SMD:R_0805_2012Metric_Pad1.20x1.40mm_HandSolder, B.Cu at (71.5, 55.9)
Routing:
- net VCC: track 50.5 -> 60.1 mm, vias 4 -> 5
- net RST: track 69.0 -> 78.3 mm
- net AOUT: track 65.2 -> 73.5 mm
- net UP: track 65.1 -> 72.5 mm
- net LOAD: track 57.5 -> 62.8 mm
- net Net-(D17-Pad2): track 0.00 -> 3.13 mm, vias 0 -> 1
- net Net-(D18-Pad2): track 0.00 -> 3.04 mm, vias 0 -> 1
- net Net-(D19-Pad1): track 0.00 -> 2.44 mm, vias 0 -> 1
- net ~RST~: track 61.9 -> 64.1 mm
Other:
- board text added: "Program Counter v1.0"
- board text added: "Velko 2021"
