File: hardware/pcb/flash_writer/flash_writer/flash_writer.kicad_pcb (KiCad board)
At the start: 2 copper layers, 68.6 x 53.3 mm, 20 parts, among them P1 Power, P2 Analog, P3 Digital, P4 Digital, P5 CONN_01X01, P6 CONN_01X01, P7 CONN_01X01, P8 CONN_01X01, U1 74HC595, U2 74HC595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

Commit message: Add CE control
Parts:
- added R4: 10K, Resistor_SMD:R_0805_2012Metric_Pad1.20x1.40mm_HandSolder, F.Cu at (161.8, 120.0)
Connections:
- P2 pad 1: (no net) -> ~CE~
- U3 pad 22: GND -> ~CE~
Routing:
- net ~CE~: track 0.00 -> 44.5 mm, vias 0 -> 1
- net +5V: track 39.9 -> 51.6 mm
- net GND: track 32.3 -> 30.9 mm, vias 12 -> 11
Other:
- board text added: "* SST39SF010 * SST39SF020 * SST39SF040"
- board text removed: "* SST39SF1010 * SST39SF1020 * SST39SF1040"

Commit message: Writer finishing touches
Changed lines of the file:
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@@
     (visible_elements 7FFFFFFF)
     (pcbplotparams
-      (layerselection 0x00030_80000001)
-      (usegerberextensions false)
-      (usegerberattributes true)
-      (usegerberadvancedattributes true)
-      (creategerberjobfile true)
+      (layerselection 0x010fc_ffffffff)
+      (usegerberextensions true)
+      (usegerberattributes false)
+      (usegerberadvancedattributes false)
+      (creategerberjobfile false)
       (excludeedgelayer true)
       (linewidth 0.100000)
@@
       (plotinvisibletext false)
       (padsonsilk false)
-      (subtractmaskfromsilk false)
+      (subtractmaskfromsilk true)
       (outputformat 1)
       (mirror false)
-      (drillshape 1)
+      (drillshape 0)
       (scaleselection 1)
-      (outputdirectory ""))
+      (outputdirectory "flw_gerbers/"))
   )
   (net 0 "")
@@
       (effects (font (size 1 1) (thickness 0.15)))
     )
-    (fp_text value 10K (at 0 1.65 90) (layer F.SilkS)
-      (effects (font (size 1 1) (thickness 0.15)))
-    )
-    (fp_text user %R (at 0 0 90) (layer F.Fab)
-      (effects (font (size 0.5 0.5) (thickness 0.08)))
+    (fp_text value 10K (at 0 1.65 90 unlocked) (layer F.SilkS)
+      (effects (font (size 1 1) (thickness 0.15)))
     )
     (fp_line (start -1 0.625) (end -1 -0.625) (layer F.Fab) (width 0.1))
@@
     (fp_line (start 1.85 -0.95) (end 1.85 0.95) (layer F.CrtYd) (width 0.05))
     (fp_line (start 1.85 0.95) (end -1.85 0.95) (layer F.CrtYd) (width 0.05))
-    (pad 2 smd roundrect (at 1 0 270) (size 1.2 1.4) (layers F.Cu F.Paste F.Mask) (roundrect_rratio 0.208333)
+    (fp_text user %R (at 0 0 90) (layer F.Fab)
+      (effects (font (size 0.5 0.5) (thickness 0.08)))
+    )
+    (pad 2 smd roundrect (at 1 0 270) (size 1.2 1.4) (layers F.Cu F.Paste F.Mask) (roundrect_rratio 0.2083325)
       (net 38 ~CE~))
-    (pad 1 smd roundrect (at -1 0 270) (size 1.2 1.4) (layers F.Cu F.Paste F.Mask) (roundrect_rratio 0.208333)
+    (pad 1 smd roundrect (at -1 0 270) (size 1.2 1.4) (layers F.Cu F.Paste F.Mask) (roundrect_rratio 0.2083325)
       (net 1 +5V))
     (model ${KISYS3DMOD}/Resistor_SMD.3dshapes/R_0805_2012Metric.wrl
@@
       (effects (font (size 1 1) (thickness 0.15)))
     )
-    (fp_text value 74HC595 (at 0 5.9 90) (layer F.Fab)
+    (fp_text value 74HC595 (at 0 0 180 unlocked) (layer F.SilkS)
       (effects (font (size 1 1) (thickness 0.15)))
     )
@@
       (effects (font (size 1 1) (thickness 0.15)))
     )
-    (fp_text value 74HC595 (at 0 5.9) (layer F.Fab)
+    (fp_text value 74HC595 (at 0 -0.0635 90) (layer F.SilkS)
       (effects (font (size 1 1) (thickness 0.15)))
     )
@@
       (effects (font (size 1 1) (thickness 0.15)))
     )
-    (fp_text value 74HC595 (at 0 5.9) (layer F.Fab)
+    (fp_text value 74HC595 (at 0 0 90) (layer F.SilkS)
       (effects (font (size 1 1) (thickness 0.15)))
     )
@@
       (effects (font (size 1 1) (thickness 0.15)))
     )
-    (fp_text value 10K (at 2.683 -0.127 180) (layer F.SilkS)
+    (fp_text value 10K (at 2.683 -0.127 180 unlocked) (layer F.SilkS)
       (effects (font (size 1 1) (thickness 0.15)))
     )
@@
       (effects (font (size 0.5 0.5) (thickness 0.08)))
     )
-    (pad 2 smd roundrect (at 1 0 270) (size 1.2 1.4) (layers F.Cu F.Paste F.Mask) (roundrect_rratio 0.208333)
-      (net 2 GND))
-    (pad 1 smd roundrect (at -1 0 270) (size 1.2 1.4) (layers F.Cu F.Paste F.Mask) (roundrect_rratio 0.208333)
+    (pad 2 smd roundrect (at 1 0 270) (size 1.2 1.4) (layers F.Cu F.Paste F.Mask) (roundrect_rratio 0.2083325)
+      (net 2 GND))
+    (pad 1 smd roundrect (at -1 0 270) (size 1.2 1.4) (layers F.Cu F.Paste F.Mask) (roundrect_rratio 0.2083325)
       (net 7 MISO))
     (model ${KISYS3DMOD}/Resistor_SMD.3dshapes/R_0805_2012Metric.wrl
@@
       (effects (font (size 0.5 0.5) (thickness 0.08)))
     )
-    (pad 2 smd roundrect (at 1 0 90) (size 1.2 1.4) (layers F.Cu F.Paste F.Mask) (roundrect_rratio 0.208333)
+    (pad 2 smd roundrect (at 1 0 90) (size 1.2 1.4) (layers F.Cu F.Paste F.Mask) (roundrect_rratio 0.2083325)
       (net 10 ~WE~))
-    (pad 1 smd roundrect (at -1 0 90) (size 1.2 1.4) (layers F.Cu F.Paste F.Mask) (roundrect_rratio 0.208333)
+    (pad 1 smd roundrect (at -1 0 90) (size 1.2 1.4) (layers F.Cu F.Paste F.Mask) (roundrect_rratio 0.2083325)
       (net 1 +5V))
     (model ${KISYS3DMOD}/Resistor_SMD.3dshapes/R_0805_2012Metric.wrl
@@
       (effects (font (size 1 1) (thickness 0.15)))
     )
-    (fp_text value 10K (at -2.81 -1.27) (layer F.SilkS)
+    (fp_text value 10K (at -2.81 -1.27 180 unlocked) (layer F.SilkS)
       (effects (font (size 1 1) (thickness 0.15)))
     )
@@
       (effects (font (size 0.5 0.5) (thickness 0.08)))
     )
-    (pad 2 smd roundrect (at 1 0 90) (size 1.2 1.4) (layers F.Cu F.Paste F.Mask) (roundrect_rratio 0.208333)
+    (pad 2 smd roundrect (at 1 0 90) (size 1.2 1.4) (layers F.Cu F.Paste F.Mask) (roundrect_rratio 0.2083325)
       (net 9 ~OE~))
-    (pad 1 smd roundrect (at -1 0 90) (size 1.2 1.4) (layers F.Cu F.Paste F.Mask) (roundrect_rratio 0.208333)
+    (pad 1 smd roundrect (at -1 0 90) (size 1.2 1.4) (layers F.Cu F.Paste F.Mask) (roundrect_rratio 0.2083325)
       (net 1 +5V))
     (model ${KISYS3DMOD}/Resistor_SMD.3dshapes/R_0805_2012Metric.wrl
@@
       (effects (font (size 1 1) (thickness 0.15)))
     )
-    (fp_text value 10uF (at 0.0215 -1.7145) (layer F.SilkS)
+    (fp_text value 10uF (at 0.0215 -1.7145 180 unlocked) (layer F.SilkS)
       (effects (font (size 1 1) (thickness 0.15)))
     )
@@
       (effects (font (size 0.5 0.5) (thickness 0.08)))
     )
-    (pad 2 smd roundrect (at 1.0375 0) (size 1.175 1.45) (layers F.Cu F.Paste F.Mask) (roundrect_rratio 0.212766)
-      (net 2 GND))
-    (pad 1 smd roundrect (at -1.0375 0) (size 1.175 1.45) (layers F.Cu F.Paste F.Mask) (roundrect_rratio 0.212766)
+    (pad 2 smd roundrect (at 1.0375 0) (size 1.175 1.45) (layers F.Cu F.Paste F.Mask) (roundrect_rratio 0.2127659574468085)
+      (net 2 GND))
+    (pad 1 smd roundrect (at -1.0375 0) (size 1.175 1.45) (layers F.Cu F.Paste F.Mask) (roundrect_rratio 0.2127659574468085)
       (net 1 +5V))
     (model ${KISYS3DMOD}/Capacitor_SMD.3dshapes/C_0805_2012Metric.wrl
@@
       (effects (font (size 0.5 0.5) (thickness 0.08)) (justify mirror))
     )
-    (pad 2 smd roundrect (at 1.0375 0 90) (size 1.175 1.45) (layers B.Cu B.Paste B.Mask) (roundrect_rratio 0.212766)
-      (net 2 GND))
-    (pad 1 smd roundrect (at -1.0375 0 90) (size 1.175 1.45) (layers B.Cu B.Paste B.Mask) (roundrect_rratio 0.212766)
+    (pad 2 smd roundrect (at 1.0375 0 90) (size 1.175 1.45) (layers B.Cu B.Paste B.Mask) (roundrect_rratio 0.2127659574468085)
+      (net 2 GND))
+    (pad 1 smd roundrect (at -1.0375 0 90) (size 1.175 1.45) (layers B.Cu B.Paste B.Mask) (roundrect_rratio 0.2127659574468085)
       (net 1 +5V))
     (model ${KISYS3DMOD}/Capacitor_SMD.3dshapes/C_0805_2012Metric.wrl
@@
       (effects (font (size 0.5 0.5) (thickness 0.08)))
     )
-    (pad 2 smd roundrect (at 1.0375 0) (size 1.175 1.45) (layers F.Cu F.Paste F.Mask) (roundrect_rratio 0.212766)
-      (net 2 GND))
-    (pad 1 smd roundrect (at -1.0375 0) (size 1.175 1.45) (layers F.Cu F.Paste F.Mask) (roundrect_rratio 0.212766)
+    (pad 2 smd roundrect (at 1.0375 0) (size 1.175 1.45) (layers F.Cu F.Paste F.Mask) (roundrect_rratio 0.2127659574468085)
+      (net 2 GND))
+    (pad 1 smd roundrect (at -1.0375 0) (size 1.175 1.45) (layers F.Cu F.Paste F.Mask) (roundrect_rratio 0.2127659574468085)
       (net 1 +5V))
     (model ${KISYS3DMOD}/Capacitor_SMD.3dshapes/C_0805_2012Metric.wrl
@@
       (effects (font (size 0.5 0.5) (thickness 0.08)))
     )
-    (pad 2 smd roundrect (at 1.0375 0 270) (size 1.175 1.45) (layers F.Cu F.Paste F.Mask) (roundrect_rratio 0.212766)
-      (net 2 GND))
-    (pad 1 smd roundrect (at -1.0375 0 270) (size 1.175 1.45) (layers F.Cu F.Paste F.Mask) (roundrect_rratio 0.212766)
+    (pad 2 smd roundrect (at 1.0375 0 270) (size 1.175 1.45) (layers F.Cu F.Paste F.Mask) (roundrect_rratio 0.2127659574468085)
+      (net 2 GND))
+    (pad 1 smd roundrect (at -1.0375 0 270) (size 1.175 1.45) (layers F.Cu F.Paste F.Mask) (roundrect_rratio 0.2127659574468085)
       (net 1 +5V))
     (model ${KISYS3DMOD}/Capacitor_SMD.3dshapes/C_0805_2012Metric.wrl
@@
       (effects (font (size 0.5 0.5) (thickness 0.08)))
     )
-    (pad 2 smd roundrect (at 1.0375 0 180) (size 1.175 1.45) (layers F.Cu F.Paste F.Mask) (roundrect_rratio 0.212766)
-      (net 2 GND))
-    (pad 1 smd roundrect (at -1.0375 0 180) (size 1.175 1.45) (layers F.Cu F.Paste F.Mask) (roundrect_rratio 0.212766)
+    (pad 2 smd roundrect (at 1.0375 0 180) (size 1.175 1.45) (layers F.Cu F.Paste F.Mask) (roundrect_rratio 0.2127659574468085)
+      (net 2 GND))
+    (pad 1 smd roundrect (at -1.0375 0 180) (size 1.175 1.45) (layers F.Cu F.Paste F.Mask) (roundrect_rratio 0.2127659574468085)
       (net 1 +5V))
     (model ${KISYS3DMOD}/Capacitor_SMD.3dshapes/C_0805_2012Metric.wrl
