File: hardware/pcb/alu_back/alu_back.kicad_pcb (KiCad board)
At the start: 2 copper layers, 132.1 x 114.3 mm, 31 parts, among them J1 SYNC, J2 BUS, J3 FLAGS, J4 OUT, J5 FCTL, J6 LOAD, J7 ARGS, J8 POWER, U1 Register A, U10 74HC125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

Commit message: Fix ALU input selector
Parts:
- U10: footprint Package_SO:SO-14_3.9x8.65mm_P1.27mm -> Package_SO:SOIC-14_3.9x8.7mm_P1.27mm
- U12, U13: footprint Package_SO:SO-16_3.9x9.9mm_P1.27mm -> Package_SO:SOIC-16_3.9x9.9mm_P1.27mm
Connections:
- net ARG_AB renamed ARG_AR
- net ARG_BB renamed ARG_BR
- net ARG_CB renamed ARG_CR
- net ARG_DB renamed ARG_DR
- J7 pad 1: Net-(J7-Pad1) -> (no net)
- J7 pad 2: Net-(J7-Pad2) -> (no net)
- J7 pad 4: ARG_B2 -> ARG_R2
- J7 pad 5: ARG_B1 -> ARG_R1
- J7 pad 6: ARG_B0 -> ARG_R0
- J7 pad 7: ARG_A1 -> ARG_L1
- J7 pad 8: ARG_A0 -> ARG_L0
- U1 pad 3: ARG_AA -> ARG_AL
- U11 pad 19: ARG_B2 -> ARG_ZR
- U12 pad 1: ARG_A0 -> ARG_R0
- U12 pad 10: Net-(U12-Pad10) -> (no net)
- U12 pad 11: Net-(U12-Pad11) -> (no net)
- U12 pad 2: ARG_A1 -> ARG_R1
- U12 pad 3: GND -> ARG_R2
- U12 pad 7: Net-(U12-Pad7) -> (no net)
- U12 pad 9: Net-(U12-Pad9) -> ARG_ZR
- U13 pad 1: ARG_B0 -> ARG_L0
- U13 pad 10: ARG_BA -> (no net)
- U13 pad 11: ARG_AA -> (no net)
- U13 pad 12: Net-(U13-Pad12) -> ARG_DL
- U13 pad 13: Net-(U13-Pad13) -> ARG_CL
- U13 pad 14: Net-(U13-Pad14) -> ARG_BL
- U13 pad 15: Net-(U13-Pad15) -> ARG_AL
- U13 pad 2: ARG_B1 -> ARG_L1
- U13 pad 3: ARG_B2 -> GND
- U13 pad 7: ARG_DA -> (no net)
- U13 pad 9: ARG_CA -> (no net)
- U2 pad 3: ARG_BA -> ARG_BL
- U3 pad 3: ARG_CA -> ARG_CL
- U4 pad 3: ARG_DA -> ARG_DL
- U5 pad 3: Net-(U5-Pad3) -> (no net)
- U5 pad 4: Net-(U5-Pad4) -> (no net)
- U6 pad 3: Net-(U6-Pad3) -> (no net)
- U6 pad 4: Net-(U6-Pad4) -> (no net)
- U7 pad 3: Net-(U7-Pad3) -> (no net)
- U7 pad 4: Net-(U7-Pad4) -> (no net)
- U8 pad 3: Net-(U8-Pad3) -> (no net)
- U8 pad 4: Net-(U8-Pad4) -> (no net)
Routing:
- net ARG_B2: track 181.3 -> 0.00 mm, vias 3 -> 0
- net ARG_ZR: track 0.00 -> 119.3 mm
- net ARG_DA: track 59.0 -> 0.00 mm
- net ARG_L0: track 0.00 -> 57.9 mm, vias 0 -> 1
- net ARG_L1: track 0.00 -> 57.7 mm, vias 0 -> 1
- net ARG_DL: track 0.00 -> 53.9 mm
- net ARG_B0: track 44.4 -> 0.00 mm, vias 1 -> 0
- net ARG_B1: track 42.0 -> 0.00 mm, vias 1 -> 0
- net ARG_CA: track 29.5 -> 0.00 mm
- net ARG_CL: track 0.00 -> 29.4 mm
- net ARG_R2: track 0.00 -> 24.3 mm, vias 0 -> 1
- net ARG_R1: track 0.00 -> 23.4 mm, vias 0 -> 1
- net ARG_R0: track 0.00 -> 22.1 mm, vias 0 -> 1
- net VCC: track 20.3 -> 40.5 mm, vias 8 -> 10
- net ARG_AL: track 0.00 -> 19.4 mm
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Other:
- board text added: "ALU Backplane v1.1"
- board text removed: "ALU Backplane v1.0"

Commit message: Renamed ALU ARG nets (A->L, B->R)
Connections:
- net /A0 renamed /L0
- net /A1 renamed /L1
- net /A2 renamed /L2
- net /A3 renamed /L3
- net /A4 renamed /L4
- net /A5 renamed /L5
- net /A6 renamed /L6
- net /A7 renamed /L7
- net /B0 renamed /R0
- net /B1 renamed /R1
- net /B2 renamed /R2
- net /B3 renamed /R3
- net /B4 renamed /R4
- net /B5 renamed /R5
- net /B6 renamed /R6
- net /B7 renamed /R7
