File: hardware/pcb/transfer/transfer.kicad_pcb (KiCad board)
At the start: 4 copper layers, 62.2 x 21.6 mm, 48 parts, among them J2 Control, J3 Sync, J4 + Power -, J5 Address Bus, J6 Main Bus, U1 74HC173, U2 74HC157, U3 74HC245, U4 74HC173, U5 74HC157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

Commit message: Transfer register fixes
Fixes #8
Additional jumper for LOW
Wider power tracks
Parts:
- added JP2: L, Jumper:SolderJumper-2_P1.3mm_Open_RoundedPad1.0x1.5mm, B.Cu at (94.8, 48.9)
- JP1: value L -> LOW
- moved JP1 0.96 mm to (94.8, 46.4), turned to 0 degrees
Connections:
- J5 pad 15: ABUS1 -> Net-(J5-Pad15)
- U2 pad 1: MLOAD -> ALOAD
- U5 pad 1: MLOAD -> ALOAD
Routing:
- net MLOAD: track 61.4 -> 9.15 mm, vias 3 -> 0
- net ALOAD: track 28.2 -> 79.5 mm, vias 0 -> 4
- net Net-(J5-Pad15): track 0.00 -> 13.4 mm, vias 0 -> 1
- net MOUT: track 68.0 -> 76.8 mm
- net Net-(J5-Pad16): track 11.3 -> 8.49 mm, vias 0 -> 1
- net VCC: track 34.0 -> 31.4 mm
- net ABUS1: track 40.9 -> 43.0 mm
Other:
- net class Power added: clearance 0.2, trace_width 0.4, via_dia 0.8, via_drill 0.4
- board text added: "Velko 2022"
- board text added: "v1.1"
- board text removed: "Velko 2021"
- board text removed: "v1.0"
